File: Sofle_Pico/PCB/Sofle_Pico.kicad_sch (KiCad schematic)
At the start: 116 parts, among them J1 Conn_01x05, J2 MJ-4PP-9, J3 Conn_01x04, J4 Conn_01x04, J5 Conn_02x05_Odd_Even, J7 Conn_01x04, Q1 Si2301CDS, SW1 SW_PUSH, SW10 SW_PUSH, SW11 SW_PUSH, SW12 SW_PUSH, SW13 SW_PUSH, SW14 SW_PUSH, SW15 SW_PUSH, SW16 SW_PUSH, SW17 SW_PUSH, SW18 SW_PUSH, SW19 SW_PUSH, SW2 SW_PUSH, SW20 SW_PUSH, SW21 SW_PUSH, SW22 SW_PUSH, SW23 SW_PUSH, SW24 SW_PUSH, SW25 Rotary_Encoder_Switch-Device, SW26 SW_PUSH, SW27 SW_PUSH, SW28 SW_PUSH, SW29 SW_PUSH, SW3 SW_PUSH, SW30 SW_PUSH, SW4 SW_PUSH, SW5 SW_PUSH, SW6 SW_PUSH, SW7 SW_PUSH, SW8 SW_PUSH, SW9 SW_PUSH, U2 Pico

Commit message: MX back conversion completed, passes DRC
Parts:
- SW1, SW10, SW11, SW12, SW13, SW14, SW15, SW16, SW17, SW18, SW19, SW2, SW20, SW21, SW22, SW23, SW24, SW26, SW27, SW28, SW29, SW3, SW30, SW4, SW5, SW6, SW7, SW8, SW9: footprint Sofle_Pico:SW_MX_HS_DS_1u -> Sofle_Pico:Cherry_MX_DS_Hotswap_v3.5.4
Changed lines of the file:
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@@
 			)
 		)
-		(property "Footprint" "Sofle_Pico:SW_MX_HS_DS_1u"
+		(property "Footprint" "Sofle_Pico:Cherry_MX_DS_Hotswap_v3.5.4"
 			(at 152.4 83.82 0)
 			(effects
@@
 			)
 		)
-		(property "Footprint" "Sofle_Pico:SW_MX_HS_DS_1u"
+		(property "Footprint" "Sofle_Pico:Cherry_MX_DS_Hotswap_v3.5.4"
 			(at 172.72 83.82 0)
 			(effects
@@
 			)
 		)
-		(property "Footprint" "Sofle_Pico:SW_MX_HS_DS_1u"
+		(property "Footprint" "Sofle_Pico:Cherry_MX_DS_Hotswap_v3.5.4"
 			(at 193.04 83.82 0)
 			(effects
@@
 			)
 		)
-		(property "Footprint" "Sofle_Pico:SW_MX_HS_DS_1u"
+		(property "Footprint" "Sofle_Pico:Cherry_MX_DS_Hotswap_v3.5.4"
 			(at 213.36 83.82 0)
 			(effects
@@
 			)
 		)
-		(property "Footprint" "Sofle_Pico:SW_MX_HS_DS_1u"
+		(property "Footprint" "Sofle_Pico:Cherry_MX_DS_Hotswap_v3.5.4"
 			(at 233.68 83.82 0)
 			(effects
@@
 			)
 		)
-		(property "Footprint" "Sofle_Pico:SW_MX_HS_DS_1u"
+		(property "Footprint" "Sofle_Pico:Cherry_MX_DS_Hotswap_v3.5.4"
 			(at 254 83.82 0)
 			(effects
@@
 			)
 		)
-		(property "Footprint" "Sofle_Pico:SW_MX_HS_DS_1u"
+		(property "Footprint" "Sofle_Pico:Cherry_MX_DS_Hotswap_v3.5.4"
 			(at 172.72 100.33 0)
 			(effects
@@
 			)
 		)
-		(property "Footprint" "Sofle_Pico:SW_MX_HS_DS_1u"
+		(property "Footprint" "Sofle_Pico:Cherry_MX_DS_Hotswap_v3.5.4"
 			(at 193.04 100.33 0)
 			(effects
@@
 			)
 		)
-		(property "Footprint" "Sofle_Pico:SW_MX_HS_DS_1u"
+		(property "Footprint" "Sofle_Pico:Cherry_MX_DS_Hotswap_v3.5.4"
 			(at 213.36 100.33 0)
 			(effects
@@
 			)
 		)
-		(property "Footprint" "Sofle_Pico:SW_MX_HS_DS_1u"
+		(property "Footprint" "Sofle_Pico:Cherry_MX_DS_Hotswap_v3.5.4"
 			(at 233.68 100.33 0)
 			(effects
@@
 			)
 		)
-		(property "Footprint" "Sofle_Pico:SW_MX_HS_DS_1u"
+		(property "Footprint" "Sofle_Pico:Cherry_MX_DS_Hotswap_v3.5.4"
 			(at 254 100.33 0)
 			(effects
@@
 			)
 		)
-		(property "Footprint" "Sofle_Pico:SW_MX_HS_DS_1u"
+		(property "Footprint" "Sofle_Pico:Cherry_MX_DS_Hotswap_v3.5.4"
 			(at 152.4 100.33 0)
 			(effects
@@
 			)
 		)
-		(property "Footprint" "Sofle_Pico:SW_MX_HS_DS_1u"
+		(property "Footprint" "Sofle_Pico:Cherry_MX_DS_Hotswap_v3.5.4"
 			(at 152.4 116.84 0)
 			(effects
@@
 			)
 		)
-		(property "Footprint" "Sofle_Pico:SW_MX_HS_DS_1u"
+		(property "Footprint" "Sofle_Pico:Cherry_MX_DS_Hotswap_v3.5.4"
 			(at 172.72 116.84 0)
 			(effects
@@
 			)
 		)
-		(property "Footprint" "Sofle_Pico:SW_MX_HS_DS_1u"
+		(property "Footprint" "Sofle_Pico:Cherry_MX_DS_Hotswap_v3.5.4"
 			(at 193.04 116.84 0)
 			(effects
@@
 			)
 		)
-		(property "Footprint" "Sofle_Pico:SW_MX_HS_DS_1u"
+		(property "Footprint" "Sofle_Pico:Cherry_MX_DS_Hotswap_v3.5.4"
 			(at 213.36 116.84 0)
 			(effects
@@
 			)
 		)
-		(property "Footprint" "Sofle_Pico:SW_MX_HS_DS_1u"
+		(property "Footprint" "Sofle_Pico:Cherry_MX_DS_Hotswap_v3.5.4"
 			(at 233.68 116.84 0)
 			(effects
@@
 			)
 		)
-		(property "Footprint" "Sofle_Pico:SW_MX_HS_DS_1u"
+		(property "Footprint" "Sofle_Pico:Cherry_MX_DS_Hotswap_v3.5.4"
 			(at 254 116.84 0)
 			(effects
@@
 			)
 		)
-		(property "Footprint" "Sofle_Pico:SW_MX_HS_DS_1u"
+		(property "Footprint" "Sofle_Pico:Cherry_MX_DS_Hotswap_v3.5.4"
 			(at 152.4 133.35 0)
 			(effects
@@
 			)
 		)
-		(property "Footprint" "Sofle_Pico:SW_MX_HS_DS_1u"
+		(property "Footprint" "Sofle_Pico:Cherry_MX_DS_Hotswap_v3.5.4"
 			(at 170.18 149.86 0)
 			(effects
@@
 			)
 		)
-		(property "Footprint" "Sofle_Pico:SW_MX_HS_DS_1u"
+		(property "Footprint" "Sofle_Pico:Cherry_MX_DS_Hotswap_v3.5.4"
 			(at 233.68 149.86 0)
 			(effects
@@
 			)
 		)
-		(property "Footprint" "Sofle_Pico:SW_MX_HS_DS_1u"
+		(property "Footprint" "Sofle_Pico:Cherry_MX_DS_Hotswap_v3.5.4"
 			(at 172.72 133.35 0)
 			(effects
@@
 			)
 		)
-		(property "Footprint" "Sofle_Pico:SW_MX_HS_DS_1u"
+		(property "Footprint" "Sofle_Pico:Cherry_MX_DS_Hotswap_v3.5.4"
 			(at 233.68 133.35 0)
 			(effects
@@
 			)
 		)
-		(property "Footprint" "Sofle_Pico:SW_MX_HS_DS_1u"
+		(property "Footprint" "Sofle_Pico:Cherry_MX_DS_Hotswap_v3.5.4"
 			(at 254 149.86 0)
 			(effects
@@
 			)
 		)
-		(property "Footprint" "Sofle_Pico:SW_MX_HS_DS_1u"
+		(property "Footprint" "Sofle_Pico:Cherry_MX_DS_Hotswap_v3.5.4"
 			(at 193.04 133.35 0)
 			(effects
@@
 			)
 		)
-		(property "Footprint" "Sofle_Pico:SW_MX_HS_DS_1u"
+		(property "Footprint" "Sofle_Pico:Cherry_MX_DS_Hotswap_v3.5.4"
 			(at 254 133.35 0)
 			(effects
@@
 			)
 		)
-		(property "Footprint" "Sofle_Pico:SW_MX_HS_DS_1u"
+		(property "Footprint" "Sofle_Pico:Cherry_MX_DS_Hotswap_v3.5.4"
 			(at 213.36 133.35 0)
 			(effects
@@
 			)
 		)
-		(property "Footprint" "Sofle_Pico:SW_MX_HS_DS_1u"
+		(property "Footprint" "Sofle_Pico:Cherry_MX_DS_Hotswap_v3.5.4"
 			(at 213.36 149.86 0)
 			(effects
@@
 			)
 		)
-		(property "Footprint" "Sofle_Pico:SW_MX_HS_DS_1u"
+		(property "Footprint" "Sofle_Pico:Cherry_MX_DS_Hotswap_v3.5.4"
 			(at 193.04 149.86 0)
 			(effects

Commit message: Final  layout and silk gloss effort
Passes DRCs

Gerbers generated
Other:
- note added: "OPTIONAL: Split Master Assignment Install Resistor value ~2.2-10k R4 3.3V = LEFT R3 GND = RIGHT"
- note removed: "OPTIONAL: Split Hand Designation 3.3V = LEFT GND = RIGHT"
Changed lines of the file:
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@@
+		)
+	)
+	(text "OPTIONAL:\nSplit Master Assignment\nInstall Resistor value ~2.2-10k\nR4 3.3V = LEFT\nR3 GND = RIGHT"
+		(exclude_from_sim no)
+		(at 105.156 76.708 0)
+		(effects
+			(font
+				(size 1.27 1.27)
+			)
+			(justify left bottom)
 		)
 	)
@@
 		(effects
 			(font
-				(size 1.27 1.27)
-			)
-			(justify left bottom)
-		)
-	)
-	(text "OPTIONAL:\nSplit Hand Designation\n3.3V = LEFT\nGND = RIGHT"
-		(exclude_from_sim no)
-		(at 102.87 74.93 0)
-		(effects
-			(font
