File: Sofle_Pico_Choc/PCB/Sofle_Pico_Choc.kicad_sch (KiCad schematic)
At the start: 116 parts, among them J1 Conn_01x05, J2 MJ-4PP-9, J3 Conn_01x04, J4 Conn_01x04, J5 Conn_02x05_Odd_Even, J7 Conn_01x04, Q1 Si2301CDS, SW1 SW_PUSH, SW10 SW_PUSH, SW11 SW_PUSH, SW12 SW_PUSH, SW13 SW_PUSH, SW14 SW_PUSH, SW15 SW_PUSH, SW16 SW_PUSH, SW17 SW_PUSH, SW18 SW_PUSH, SW19 SW_PUSH, SW2 SW_PUSH, SW20 SW_PUSH, SW21 SW_PUSH, SW22 SW_PUSH, SW23 SW_PUSH, SW24 SW_PUSH, SW25 Rotary_Encoder_Switch-Device, SW26 SW_PUSH, SW27 SW_PUSH, SW28 SW_PUSH, SW29 SW_PUSH, SW3 SW_PUSH, SW30 SW_PUSH, SW4 SW_PUSH, SW5 SW_PUSH, SW6 SW_PUSH, SW7 SW_PUSH, SW8 SW_PUSH, SW9 SW_PUSH, U2 Pico

Commit message: KiCAD 8 choc files w/ fixed logos
Parts:
- C2: value 0.1uF -> 1uF; JLCPCB_PN C49678 -> C28323; MFG YAGEO -> Samsung; MFG PN CC0805KRX7R9BB104 -> CL21B105KBFNNNE
Other:
- note added: "D31 is NOT REQUIRED for RPI Pico SCH compliant boards that have a reverse-polarity protection diode between VBUS and VSYS. VSYS voltage varies depending on protection diode voltage drop. User must verify whether their chosen MCU Module is 1:1 pin compliant with RPI Pico VSYS ≈ 4.9-5.0V with USB Power VSYS ≈ 4.7-4.9V with TRRS Power Refer to Sofle-Pico build guide and your RPI Module Datasheet/SCH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"
- note added: "OPTIONAL 0805 surface mount capacitors for power smoothing / decoupling"
- note removed: "D31 is not required for RPI Pico SCH compliant boards that have an onboard Schottky Diode. Refer to Sofle-Pico build guide and your RPI Module Datasheet/SCH. VSYS is variable depending on diode used! User MUST know/verify whether or not their MCU Module is pin compliant with RPI Pico. Read RPI Pico datasheet Chapter 4.5-4.6 VSYS≈4.9-5.0V w/ USB Power VSYS≈4.7-4.9V w/ TRRS Power"
- note removed: "OPTIONAL decoupling 0805"
- moved on the sheet: C1, C3, C4

Commit message: Final  layout and silk gloss effort
Passes DRCs

Gerbers generated
Other:
- note added: "OPTIONAL: Split Master Assignment Install Resistor value ~2.2-10k R4 3.3V = LEFT R3 GND = RIGHT"
- note removed: "OPTIONAL: Split Hand Designation 3.3V = LEFT GND = RIGHT"
Changed lines of the file:
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@@
 		)
 	)
-	(text "OPTIONAL:\nSplit Hand Designation\n3.3V = LEFT\nGND = RIGHT"
+	(text "OPTIONAL:\nSplit Master Assignment\nInstall Resistor value ~2.2-10k\nR4 3.3V = LEFT\nR3 GND = RIGHT"
 		(exclude_from_sim no)
 		(at 102.87 74.93 0)
